File: hardware/v0.2/2.sch (EAGLE design)
At the start: 26 parts, among them IC2 STM32F10XCXT6, U1 ADXL345"

Commit message: modify pcb design
Parts:
- removed R12, R13, R14, R15: 470R, rcl:R-EU_R0603
- added C3: 10uF, SparkFun-Capacitors:10UF-16V-10%(TANT)
- added LED3, LED4, LED5, LED6, LED7, LED8: (no value), SparkFun-LED:LED1206
- added R1, R2, R6, R7, R8, R9: 10K, rcl:R-EU_R0603
- added S1: SWITCH-MOMENTARY-2-SMD-1101NE, SparkFun-Electromechanical:SWITCH-MOMENTARY-2-SMD-1101NE
- LED1, LED2: value LED-TRICOLOR-5050NO_IC -> (none); device SparkFun-LED:LED-TRICOLOR-5050NO_IC -> SparkFun-LED:LED1206
- R10, R11: value 470R -> 10K
Connections:
- removed net LED1_B: LED1.BLU-C
- removed net LED1_G: LED1.GRN-C
- removed net LED1_R: LED1.RED-C
- removed net LED2_B: LED2.BLU-C
- removed net LED2_G: LED2.GRN-C
- removed net LED2_R: LED2.RED-C
- removed net N$10: LED1.GRN-A, R11.2
- removed net N$11: LED1.RED-A, R12.2
- removed net N$12: LED2.BLU-A, R13.2
- removed net N$13: LED2.GRN-A, R14.2
- removed net N$14: LED2.RED-A, R15.2
- removed net N$8: LED1.BLU-A, R10.2
- new net N$3: R6.1, R7.2
- new net N$4: R8.1, R9.2
- net 3.3V: now also C3.+, S1.1; no longer R10.1, R11.1, R12.1, R13.1, R14.1, R15.1
- net GND: now also C3.-
- net N$2: now also S1.2
Other:
- moved on the sheet: C1, C10, C11, C2, C4, C8, C9, R10, R11, R4, U1

Commit message: Updated V2 PCB design
Parts:
- removed C11: 4.7u, rcl:C-EUC0603K
- removed JP5: M02PTH, SparkFun-Connectors:M02PTH
- removed LED5, LED6, LED7, LED8: (no value), SparkFun-LED:LED1206
- added BL1: (no value), digital-toy:BL8530-XX2_RN
- added C6: 10u, rcl:C-EUC0603K
- added C7: 0.1u, rcl:C-EUC0603K
- added D1: BAT20JFILM, SparkFun-DiscreteSemi:BAT20JFILM
- added JP3: (no value), SparkFun-Connectors:M04PTH
- added L1: (no value), SparkFun-Passives:INDUCTORVLF4012A
- C1, C2: value 0.1u -> 10uF; device rcl:C-EUC0603K -> SparkFun-Capacitors:10UF-16V-10%(TANT)
- C10: value 0.1u -> 4.7u
- C3, C4: value 10uF -> 0.1u; device SparkFun-Capacitors:10UF-16V-10%(TANT) -> rcl:C-EUC0603K
- C5: value 10u -> 100uF; device rcl:C-EUC0603K -> SparkFun-Capacitors:47UF-TANT
- JP1: device SparkFun-Connectors:M04PTH -> SparkFun-Connectors:M03PTH
- JP4: value (none) -> M02PTH; device SparkFun-Connectors:M03PTH -> SparkFun-Connectors:M02PTH
- LED1, LED2: value (none) -> LED-TRICOLOR-5050NO_IC; device SparkFun-LED:LED1206 -> SparkFun-LED:LED-TRICOLOR-5050NO_IC
- R1, R2, R3, R4, R5, R6, R8, R9: value 10K -> 270
- renumbered IC2 to IC1
Connections:
- new net 2.8V: C1.+, C10.1, C2.+, C3.1, C4.1, C7.1, C8.1, C9.1, F1.1, IC1AN_POWER.VBAT, IC1AN_POWER.VDDA, IC1POWER.VDD_1, IC1POWER.VDD_2, IC1POWER.VDD_3, JP3.1, JP4.1, L1.1, R11.1, S1.1, U1.VDD, U1.VS
- new net LED1_B: LED1.BLU-C
- new net LED1_G: LED1.GRN-C
- new net LED1_R: LED1.RED-C
- new net LED2_B: LED2.BLU-C
- new net LED2_G: LED2.GRN-C
- new net LED2_R: LED2.RED-C
- new net LED_EN: BL1.CE
- new net N$10: LED2.GRN-A, R5.2
- new net N$11: LED2.RED-A, R6.2
- new net N$12: BL1.LX, D1.A, L1.2
- new net N$6: LED1.BLU-A, R1.2
- new net N$7: LED1.GRN-A, R2.2
- new net N$8: LED1.RED-A, R3.2
- new net N$9: LED2.BLU-A, R4.2
- net 3.3V: now also BL1.OUT, C5.+, D1.C, R1.1, R2.1, R4.1, R5.1, R6.1, R8.1, R9.1; no longer C1.1, C10.1, C11.1, C2.1, C3.+, C4.+, C8.1, C9.1, F1.1, IC1AN_POWER.VBAT, IC1AN_POWER.VDDA, IC1POWER.VDD_1, IC1POWER.VDD_2, IC1POWER.VDD_3, JP1.1, JP5.1, S1.1, U1.VDD
- net BOOT0: now also JP4.2, R7.2; no longer JP5.2, R5.2
- net GND: now also BL1.GND, C1.-, C2.-, C3.2, C4.2, C5.-, C6.2, C7.2, JP1.3, JP3.4, R10.2, R7.1; no longer C1.2, C11.2, C2.2, C3.-, C4.-, C5.2, JP1.4, JP4.3, R4.2, R5.1
- net N$2: now also R10.1; no longer R4.1
- net N$3: now also LED4.A, R9.2; no longer R6.1, R7.2
- net N$4: now also LED3.A, R8.2; no longer R8.1, R9.2
- net RESET: now also C6.1, R11.2; no longer C5.1, R3.2
- net SWCLK: now also JP3.3; no longer JP1.3
- net SWDIO: now also JP3.2; no longer JP1.2
- net USART1_RX: now also JP1.2; no longer JP4.2
- net USART1_TX: now also JP1.1; no longer JP4.1
Other:
- moved on the sheet: C10, C8, C9, LED3, LED4, R1, R10, R11, R2, R3, R4, R5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

Commit message: update PCB design
Connections:
- removed net LED1_B: LED1.BLU-C
- removed net LED1_G: LED1.GRN-C
- removed net LED1_R: LED1.RED-C
- removed net XL345_INT: IC1PORTA_L.PA3, U1.INT1
- net 3.3V: now also LED1.BLU-A, LED1.GRN-A, LED1.RED-A; no longer R1.1, R2.1, R3.1
- net N$6: now also LED1.BLU-C, R1.1; no longer LED1.BLU-A, R1.2
- net N$7: now also LED1.GRN-C, R2.1; no longer LED1.GRN-A, R2.2
- net N$8: now also LED1.RED-C, R3.1; no longer LED1.RED-A, R3.2
- net WAKEUP: now also U1.INT1; no longer U1.INT2
- net XL345_CS: now also IC1PORTB_L.PB0; no longer IC1PORTA_L.PA4
Other:
- moved on the sheet: LED1, R1, R2, R3
Changed lines of the file:
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@@
 <instance part="C1" gate="G$1" x="15.24" y="12.7"/>
 <instance part="S1" gate="G$1" x="86.36" y="40.64"/>
-<instance part="LED1" gate="D1" x="20.32" y="-27.94" rot="MR0"/>
+<instance part="LED1" gate="D1" x="10.16" y="-27.94" rot="MR0"/>
 <instance part="LED2" gate="D1" x="20.32" y="-50.8" rot="MR0"/>
 <instance part="LED3" gate="G$1" x="63.5" y="22.86" rot="MR270"/>
@@
 <instance part="C5" gate="G$1" x="144.78" y="-71.12"/>
 <instance part="SUPPLY10" gate="G$1" x="15.24" y="20.32"/>
-<instance part="R1" gate="G$1" x="-2.54" y="-25.4"/>
-<instance part="R2" gate="G$1" x="-2.54" y="-27.94"/>
-<instance part="R3" gate="G$1" x="-2.54" y="-30.48"/>
+<instance part="R1" gate="G$1" x="33.02" y="-25.4"/>
+<instance part="R2" gate="G$1" x="33.02" y="-27.94"/>
+<instance part="R3" gate="G$1" x="33.02" y="-30.48"/>
 <instance part="R4" gate="G$1" x="-2.54" y="-48.26"/>
 <instance part="R5" gate="G$1" x="-2.54" y="-50.8"/>
@@
 </segment>
 <segment>
-<pinref part="U1" gate="G$1" pin="INT2"/>
-<wire x1="137.16" y1="-20.32" x2="154.94" y2="-20.32" width="0.1524" layer="91"/>
-<label x="139.7" y="-20.32" size="1.778" layer="95"/>
+<pinref part="U1" gate="G$1" pin="INT1"/>
+<wire x1="137.16" y1="-17.78" x2="154.94" y2="-17.78" width="0.1524" layer="91"/>
+<label x="139.7" y="-17.78" size="1.778" layer="95"/>
 </segment>
 </net>
@@
 </segment>
 <segment>
-<pinref part="IC1" gate="PORTA_L" pin="PA4"/>
-<wire x1="109.22" y1="68.58" x2="88.9" y2="68.58" width="0.1524" layer="91"/>
-<label x="91.44" y="68.58" size="1.778" layer="95"/>
+<pinref part="IC1" gate="PORTB_L" pin="PB0"/>
+<wire x1="109.22" y1="45.72" x2="88.9" y2="45.72" width="0.1524" layer="91"/>
+<label x="91.44" y="45.72" size="1.778" layer="95"/>
 </segment>
 </net>
@@
 <wire x1="109.22" y1="66.04" x2="88.9" y2="66.04" width="0.1524" layer="91"/>
 <label x="91.44" y="66.04" size="1.778" layer="95"/>
-</segment>
-</net>
-<net name="XL345_INT" class="0">
-<segment>
-<pinref part="U1" gate="G$1" pin="INT1"/>
-<wire x1="137.16" y1="-17.78" x2="154.94" y2="-17.78" width="0.1524" layer="91"/>
-<label x="139.7" y="-17.78" size="1.778" layer="95"/>
-</segment>
-<segment>
-<pinref part="IC1" gate="PORTA_L" pin="PA3"/>
-<wire x1="109.22" y1="71.12" x2="88.9" y2="71.12" width="0.1524" layer="91"/>
-<label x="91.44" y="71.12" size="1.778" layer="95"/>
 </segment>
 </net>
@@
 <pinref part="C2" gate="G$1" pin="+"/>
 <wire x1="86.36" y1="0" x2="86.36" y2="-2.54" width="0.1524" layer="91"/>
-<pinref part="C4" gate="G$1" pin="1"/>
 <wire x1="86.36" y1="-2.54" x2="86.36" y2="-5.08" width="0.1524" layer="91"/>
-<wire x1="104.14" y1="-5.08" x2="104.14" y2="-2.54" width="0.1524" layer="91"/>
-<wire x1="104.14" y1="-2.54" x2="93.98" y2="-2.54" width="0.1524" layer="91"/>
+<wire x1="114.3" y1="-2.54" x2="104.14" y2="-2.54" width="0.1524" layer="91"/>
 <junction x="86.36" y="-2.54"/>
 <pinref part="C3" gate="G$1" pin="1"/>
+<wire x1="104.14" y1="-2.54" x2="93.98" y2="-2.54" width="0.1524" layer="91"/>
 <wire x1="93.98" y1="-2.54" x2="86.36" y2="-2.54" width="0.1524" layer="91"/>
 <wire x1="93.98" y1="-5.08" x2="93.98" y2="-2.54" width="0.1524" layer="91"/>
 <junction x="93.98" y="-2.54"/>
 <pinref part="U1" gate="G$1" pin="VDD"/>
-<wire x1="104.14" y1="-2.54" x2="109.22" y2="-2.54" width="0.1524" layer="91"/>
+<pinref part="SUPPLY17" gate="G$1" pin="2.8V"/>
+<pinref part="C4" gate="G$1" pin="1"/>
+<pinref part="U1" gate="G$1" pin="VS"/>
+<wire x1="104.14" y1="-5.08" x2="114.3" y2="-5.08" width="0.1524" layer="91"/>
+<wire x1="104.14" y1="-5.08" x2="104.14" y2="-2.54" width="0.1524" layer="91"/>
+<junction x="104.14" y="-5.08"/>
 <junction x="104.14" y="-2.54"/>
-<pinref part="SUPPLY17" gate="G$1" pin="2.8V"/>
-<pinref part="U1" gate="G$1" pin="VS"/>
-<wire x1="109.22" y1="-2.54" x2="114.3" y2="-2.54" width="0.1524" layer="91"/>
-<wire x1="114.3" y1="-5.08" x2="109.22" y2="-5.08" width="0.1524" layer="91"/>
-<wire x1="109.22" y1="-5.08" x2="109.22" y2="-2.54" width="0.1524" layer="91"/>
-<junction x="109.22" y="-2.54"/>
 </segment>
 <segment>
@@
 </segment>
 </net>
-<net name="N$6" class="0">
-<segment>
-<pinref part="R1" gate="G$1" pin="2"/>
-<pinref part="LED1" gate="D1" pin="BLU-A"/>
-<wire x1="2.54" y1="-25.4" x2="5.08" y2="-25.4" width="0.1524" layer="91"/>
-</segment>
-</net>
-<net name="N$7" class="0">
-<segment>
-<pinref part="R2" gate="G$1" pin="2"/>
-<pinref part="LED1" gate="D1" pin="GRN-A"/>
-<wire x1="2.54" y1="-27.94" x2="5.08" y2="-27.94" width="0.1524" layer="91"/>
-</segment>
-</net>
-<net name="N$8" class="0">
-<segment>
-<pinref part="R3" gate="G$1" pin="2"/>
-<pinref part="LED1" gate="D1" pin="RED-A"/>
-<wire x1="2.54" y1="-30.48" x2="5.08" y2="-30.48" width="0.1524" layer="91"/>
-</segment>
-</net>
 <net name="N$9" class="0">
 <segment>
@@
 <pinref part="SUPPLY1" gate="G$1" pin="3.3V"/>
 <wire x1="-10.16" y1="-22.86" x2="-10.16" y2="-25.4" width="0.1524" layer="91"/>
-<pinref part="R3" gate="G$1" pin="1"/>
+<pinref part="LED1" gate="D1" pin="BLU-A"/>
 <wire x1="-10.16" y1="-25.4" x2="-10.16" y2="-27.94" width="0.1524" layer="91"/>
 <wire x1="-10.16" y1="-27.94" x2="-10.16" y2="-30.48" width="0.1524" layer="91"/>
-<wire x1="-10.16" y1="-30.48" x2="-7.62" y2="-30.48" width="0.1524" layer="91"/>
-<pinref part="R2" gate="G$1" pin="1"/>
-<wire x1="-7.62" y1="-27.94" x2="-10.16" y2="-27.94" width="0.1524" layer="91"/>
+<wire x1="-5.08" y1="-25.4" x2="-10.16" y2="-25.4" width="0.1524" layer="91"/>
+<junction x="-10.16" y="-25.4"/>
+<pinref part="LED1" gate="D1" pin="GRN-A"/>
+<wire x1="-5.08" y1="-27.94" x2="-10.16" y2="-27.94" width="0.1524" layer="91"/>
 <junction x="-10.16" y="-27.94"/>
-<pinref part="R1" gate="G$1" pin="1"/>
-<wire x1="-7.62" y1="-25.4" x2="-10.16" y2="-25.4" width="0.1524" layer="91"/>
-<junction x="-10.16" y="-25.4"/>
+<pinref part="LED1" gate="D1" pin="RED-A"/>
+<wire x1="-5.08" y1="-30.48" x2="-10.16" y2="-30.48" width="0.1524" layer="91"/>
 </segment>
 <segment>
@@
 </segment>
 </net>
-<net name="LED1_B" class="0">
-<segment>
-<pinref part="LED1" gate="D1" pin="BLU-C"/>
-<wire x1="35.56" y1="-25.4" x2="48.26" y2="-25.4" width="0.1524" layer="91"/>
-<label x="38.1" y="-25.4" size="1.778" layer="95"/>
-</segment>
-</net>
-<net name="LED1_G" class="0">
-<segment>
-<pinref part="LED1" gate="D1" pin="GRN-C"/>
-<wire x1="35.56" y1="-27.94" x2="48.26" y2="-27.94" width="0.1524" layer="91"/>
-<label x="38.1" y="-27.94" size="1.778" layer="95"/>
-</segment>
-</net>
-<net name="LED1_R" class="0">
-<segment>
-<pinref part="LED1" gate="D1" pin="RED-C"/>
-<wire x1="35.56" y1="-30.48" x2="45.72" y2="-30.48" width="0.1524" layer="91"/>
-<label x="38.1" y="-30.48" size="1.778" layer="95"/>
-</segment>
-</net>
 <net name="LED2_B" class="0">
 <segment>
@@
 </segment>
 </net>
+<net name="N$6" class="0">
+<segment>
+<pinref part="R1" gate="G$1" pin="1"/>
+<pinref part="LED1" gate="D1" pin="BLU-C"/>
+<wire x1="27.94" y1="-25.4" x2="25.4" y2="-25.4" width="0.1524" layer="91"/>
+</segment>
+</net>
+<net name="N$7" class="0">
+<segment>
+<pinref part="R2" gate="G$1" pin="1"/>
+<pinref part="LED1" gate="D1" pin="GRN-C"/>
+<wire x1="27.94" y1="-27.94" x2="25.4" y2="-27.94" width="0.1524" layer="91"/>
+</segment>
+</net>
+<net name="N$8" class="0">
+<segment>
+<pinref part="R3" gate="G$1" pin="1"/>
+<pinref part="LED1" gate="D1" pin="RED-C"/>
+<wire x1="27.94" y1="-30.48" x2="25.4" y2="-30.48" width="0.1524" layer="91"/>
+</segment>
+</net>
