File: hardware/v0.2/2.sch (EAGLE design)
At the start: 36 parts, among them IC1 STM32F10XCXT6, U1 ADXL345"

Commit message: nearly finish PCB design
Connections:
- removed net XL345_INT: IC1PORTA_L.PA3, U1.INT1
- new net LED3: IC1PORTA_L.PA2, LED3.C
- new net LED4: IC1PORTB_H.PB15, LED4.C
- new net N$13: IC1PORTB_L.PB1
- net 3.3V: now also LED1.BLU-A, LED1.GRN-A, LED1.RED-A; no longer R1.1, R2.1, R3.1
- net LED1_B: now also IC1PORTB_H.PB14, R1.2; no longer LED1.BLU-C
- net LED1_G: now also IC1PORTB_H.PB12, R2.2; no longer LED1.GRN-C
- net LED1_R: now also IC1PORTB_H.PB13, R3.2; no longer LED1.RED-C
- net LED2_B: now also IC1PORTB_L.PB5
- net LED2_G: now also IC1PORTB_L.PB7
- net LED2_R: now also IC1PORTB_L.PB6
- net N$6: now also LED1.BLU-C, R1.1; no longer LED1.BLU-A, R1.2
- net N$7: now also LED1.GRN-C, R2.1; no longer LED1.GRN-A, R2.2
- net N$8: now also LED1.RED-C, R3.1; no longer LED1.RED-A, R3.2
- net WAKEUP: now also U1.INT1; no longer U1.INT2
- net XL345_CS: now also IC1PORTB_L.PB0; no longer IC1PORTA_L.PA4
Other:
- moved on the sheet: LED1, R1, R10, R2, R3

Commit message: finish version 0.2 pcb design
Parts:
- C1: value 10uF -> 22uF
- L1: value (none) -> 22uh
- renumbered BL1 to IC3, U1 to IC2
Connections:
- removed net N$13: IC1PORTB_L.PB1
- net LED2_B: now also IC1PORTB_L.PB4; no longer IC1PORTB_L.PB5
- net LED3: now also IC1PORTB_H.PB8; no longer IC1PORTA_L.PA2
- net LED_EN: now also IC1PORTA_L.PA3
Changed lines of the file:
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@@
 <part name="JP3" library="SparkFun-Connectors" deviceset="M04" device="PTH"/>
 <part name="GND1" library="SparkFun-Aesthetics" deviceset="GND" device=""/>
-<part name="U1" library="SparkFun-Sensors" deviceset="ADXL345" device="&quot;"/>
+<part name="IC2" library="SparkFun-Sensors" deviceset="ADXL345" device="&quot;"/>
 <part name="C4" library="rcl" deviceset="C-EU" device="C0603K" value="0.1u"/>
 <part name="C3" library="rcl" deviceset="C-EU" device="C0603K" value="0.1u"/>
@@
 <part name="GND2" library="SparkFun-Aesthetics" deviceset="GND" device=""/>
 <part name="GND8" library="SparkFun-Aesthetics" deviceset="GND" device=""/>
-<part name="C1" library="SparkFun-Capacitors" deviceset="10UF-16V-10%(TANT)" device="" value="10uF"/>
+<part name="C1" library="SparkFun-Capacitors" deviceset="10UF-16V-10%(TANT)" device="" value="22uF"/>
 <part name="S1" library="SparkFun-Electromechanical" deviceset="SWITCH-MOMENTARY-2" device="-SMD-1101NE"/>
 <part name="LED1" library="SparkFun-LED" deviceset="LED-TRICOLOR-5050" device="NO_IC"/>
@@
 <part name="R8" library="rcl" deviceset="R-EU_" device="R0603" value="270"/>
 <part name="R9" library="rcl" deviceset="R-EU_" device="R0603" value="270"/>
-<part name="BL1" library="digital-toy" deviceset="BL8530-XX2_RN" device=""/>
+<part name="IC3" library="digital-toy" deviceset="BL8530-XX2_RN" device=""/>
 <part name="C5" library="SparkFun-Capacitors" deviceset="47UF-TANT" device="" value="100uF"/>
 <part name="SUPPLY10" library="SparkFun-Aesthetics" deviceset="2.8V" device=""/>
@@
 <part name="SUPPLY3" library="SparkFun-Aesthetics" deviceset="3.3V" device=""/>
 <part name="SUPPLY4" library="SparkFun-Aesthetics" deviceset="3.3V" device=""/>
-<part name="L1" library="SparkFun-Passives" deviceset="INDUCTOR" device="VLF4012A"/>
+<part name="L1" library="SparkFun-Passives" deviceset="INDUCTOR" device="VLF4012A" value="22uh"/>
 <part name="GND11" library="SparkFun-Aesthetics" deviceset="GND" device=""/>
 <part name="SUPPLY5" library="SparkFun-Aesthetics" deviceset="2.8V" device=""/>
@@
 <instance part="JP3" gate="G$1" x="-7.62" y="48.26" rot="MR180"/>
 <instance part="GND1" gate="1" x="12.7" y="38.1"/>
-<instance part="U1" gate="G$1" x="124.46" y="-12.7"/>
+<instance part="IC2" gate="G$1" x="124.46" y="-12.7"/>
 <instance part="C4" gate="G$1" x="104.14" y="-7.62"/>
 <instance part="C3" gate="G$1" x="93.98" y="-7.62"/>
@@
 <instance part="GND8" gate="1" x="86.36" y="-22.86"/>
 <instance part="C1" gate="G$1" x="15.24" y="12.7"/>
-<instance part="S1" gate="G$1" x="86.36" y="40.64"/>
+<instance part="S1" gate="G$1" x="86.36" y="40.64" smashed="yes">
+<attribute name="NAME" x="83.82" y="43.18" size="1.778" layer="95"/>
+</instance>
 <instance part="LED1" gate="D1" x="10.16" y="-27.94" rot="MR0"/>
 <instance part="LED2" gate="D1" x="20.32" y="-50.8" rot="MR0"/>
@@
 <instance part="R8" gate="G$1" x="50.8" y="22.86"/>
 <instance part="R9" gate="G$1" x="50.8" y="10.16"/>
-<instance part="BL1" gate="G$1" x="121.92" y="-71.12"/>
+<instance part="IC3" gate="G$1" x="121.92" y="-71.12"/>
 <instance part="C5" gate="G$1" x="144.78" y="-71.12"/>
 <instance part="SUPPLY10" gate="G$1" x="15.24" y="20.32"/>
@@
 <pinref part="GND2" gate="1" pin="GND"/>
 <wire x1="106.68" y1="-27.94" x2="106.68" y2="-25.4" width="0.1524" layer="91"/>
-<pinref part="U1" gate="G$1" pin="GND@2"/>
+<pinref part="IC2" gate="G$1" pin="GND@2"/>
 <wire x1="106.68" y1="-25.4" x2="106.68" y2="-22.86" width="0.1524" layer="91"/>
 <wire x1="106.68" y1="-22.86" x2="106.68" y2="-20.32" width="0.1524" layer="91"/>
 <wire x1="106.68" y1="-20.32" x2="114.3" y2="-20.32" width="0.1524" layer="91"/>
-<pinref part="U1" gate="G$1" pin="GND@4"/>
+<pinref part="IC2" gate="G$1" pin="GND@4"/>
 <wire x1="114.3" y1="-22.86" x2="106.68" y2="-22.86" width="0.1524" layer="91"/>
 <junction x="106.68" y="-22.86"/>
-<pinref part="U1" gate="G$1" pin="GND@5"/>
+<pinref part="IC2" gate="G$1" pin="GND@5"/>
 <wire x1="114.3" y1="-25.4" x2="106.68" y2="-25.4" width="0.1524" layer="91"/>
 <junction x="106.68" y="-25.4"/>
@@
 <segment>
 <pinref part="C5" gate="G$1" pin="-"/>
-<pinref part="BL1" gate="G$1" pin="GND"/>
+<pinref part="IC3" gate="G$1" pin="GND"/>
 <wire x1="144.78" y1="-76.2" x2="134.62" y2="-76.2" width="0.1524" layer="91"/>
 <pinref part="GND11" gate="1" pin="GND"/>
@@
 </segment>
 <segment>
-<pinref part="U1" gate="G$1" pin="INT1"/>
+<pinref part="IC2" gate="G$1" pin="INT1"/>
 <wire x1="137.16" y1="-17.78" x2="154.94" y2="-17.78" width="0.1524" layer="91"/>
 <label x="139.7" y="-17.78" size="1.778" layer="95"/>
@@
 <net name="XL345_CS" class="0">
 <segment>
-<pinref part="U1" gate="G$1" pin="CS"/>
+<pinref part="IC2" gate="G$1" pin="CS"/>
 <wire x1="137.16" y1="-2.54" x2="154.94" y2="-2.54" width="0.1524" layer="91"/>
 <label x="139.7" y="-2.54" size="1.778" layer="95"/>
@@
 <net name="XL345_MISO" class="0">
 <segment>
-<pinref part="U1" gate="G$1" pin="SDO"/>
+<pinref part="IC2" gate="G$1" pin="SDO"/>
 <wire x1="137.16" y1="-7.62" x2="154.94" y2="-7.62" width="0.1524" layer="91"/>
 <label x="139.7" y="-7.62" size="1.778" layer="95"/>
@@
 <net name="XL345_MOSI" class="0">
 <segment>
-<pinref part="U1" gate="G$1" pin="SDA"/>
+<pinref part="IC2" gate="G$1" pin="SDA"/>
 <wire x1="137.16" y1="-10.16" x2="154.94" y2="-10.16" width="0.1524" layer="91"/>
 <label x="139.7" y="-10.16" size="1.778" layer="95"/>
@@
 <net name="XL345_SCK" class="0">
 <segment>
-<pinref part="U1" gate="G$1" pin="SCL"/>
+<pinref part="IC2" gate="G$1" pin="SCL"/>
 <wire x1="137.16" y1="-12.7" x2="154.94" y2="-12.7" width="0.1524" layer="91"/>
 <label x="139.7" y="-12.7" size="1.778" layer="95"/>
@@
 <wire x1="93.98" y1="-5.08" x2="93.98" y2="-2.54" width="0.1524" layer="91"/>
 <junction x="93.98" y="-2.54"/>
-<pinref part="U1" gate="G$1" pin="VDD"/>
+<pinref part="IC2" gate="G$1" pin="VDD"/>
 <pinref part="SUPPLY17" gate="G$1" pin="2.8V"/>
 <pinref part="C4" gate="G$1" pin="1"/>
-<pinref part="U1" gate="G$1" pin="VS"/>
+<pinref part="IC2" gate="G$1" pin="VS"/>
 <wire x1="104.14" y1="-5.08" x2="114.3" y2="-5.08" width="0.1524" layer="91"/>
 <wire x1="104.14" y1="-5.08" x2="104.14" y2="-2.54" width="0.1524" layer="91"/>
@@
 <segment>
 <wire x1="137.16" y1="-55.88" x2="137.16" y2="-68.58" width="0.1524" layer="91"/>
-<pinref part="BL1" gate="G$1" pin="OUT"/>
+<pinref part="IC3" gate="G$1" pin="OUT"/>
 <wire x1="137.16" y1="-68.58" x2="134.62" y2="-68.58" width="0.1524" layer="91"/>
 <wire x1="137.16" y1="-55.88" x2="144.78" y2="-55.88" width="0.1524" layer="91"/>
@@
 <net name="N$12" class="0">
 <segment>
-<pinref part="BL1" gate="G$1" pin="LX"/>
+<pinref part="IC3" gate="G$1" pin="LX"/>
 <wire x1="109.22" y1="-68.58" x2="106.68" y2="-68.58" width="0.1524" layer="91"/>
 <wire x1="106.68" y1="-68.58" x2="106.68" y2="-55.88" width="0.1524" layer="91"/>
@@
 </segment>
 <segment>
-<pinref part="IC1" gate="PORTB_L" pin="PB5"/>
-<wire x1="109.22" y1="33.02" x2="96.52" y2="33.02" width="0.1524" layer="91"/>
-<label x="96.52" y="33.02" size="1.778" layer="95"/>
+<pinref part="IC1" gate="PORTB_L" pin="PB4"/>
+<wire x1="109.22" y1="35.56" x2="96.52" y2="35.56" width="0.1524" layer="91"/>
+<label x="96.52" y="35.56" size="1.778" layer="95"/>
 </segment>
 </net>
@@
 <net name="LED_EN" class="0">
 <segment>
-<pinref part="BL1" gate="G$1" pin="CE"/>
+<pinref part="IC3" gate="G$1" pin="CE"/>
 <wire x1="109.22" y1="-76.2" x2="86.36" y2="-76.2" width="0.1524" layer="91"/>
 <label x="86.36" y="-76.2" size="1.778" layer="95"/>
+</segment>
+<segment>
+<pinref part="IC1" gate="PORTA_L" pin="PA3"/>
+<wire x1="109.22" y1="71.12" x2="88.9" y2="71.12" width="0.1524" layer="91"/>
+<label x="91.44" y="71.12" size="1.778" layer="95"/>
 </segment>
 </net>
@@
 </segment>
 </net>
-<net name="N$13" class="0">
-<segment>
-<pinref part="IC1" gate="PORTB_L" pin="PB1"/>
-<wire x1="109.22" y1="43.18" x2="88.9" y2="43.18" width="0.1524" layer="91"/>
-</segment>
-</net>
 <net name="LED1_G" class="0">
 <segment>
@@
 </segment>
 <segment>
-<pinref part="IC1" gate="PORTA_L" pin="PA2"/>
-<wire x1="109.22" y1="73.66" x2="88.9" y2="73.66" width="0.1524" layer="91"/>
-<label x="91.44" y="73.66" size="1.778" layer="95"/>
-</segment>
-</net>
+<pinref part="IC1" gate="PORTB_H" pin="PB8"/>
+<wire x1="144.78" y1="45.72" x2="162.56" y2="45.72" width="0.1524" layer="91"/>
+<label x="147.32" y="45.72" size="1.778" layer="95"/>
+</segment>
+</net>
